Commit message: alars_captain.launch

File: vehicles/descriptions/alars_description/urdf/alars.urdf (robot description, URDF)
Before this commit: robot alars, 4 links, 3 joints
Links:
- removed link base_link
- removed link z1_base
- added link module_base_link
- added link z1_base_link
Joints:
- joint fisheye_base_joint: parent base_link -> module_base_link
- joint gimbal_base_joint: child z1_base -> z1_base_link; parent base_link -> module_base_link
- joint rope_base_joint: parent base_link -> module_base_link

Commit message: alars.urdf: added base->module for when the module is mounted elsewhere...

File: vehicles/descriptions/alars_description/urdf/alars.urdf (robot description, URDF)
Before this commit: robot alars, 4 links, 3 joints
Links:
- removed link module_base_link
- added link alars_module_base_link
- added link base_link
- added link fisheye_camera_link
Joints:
- added joint base_to_module_joint: type fixed, parent base_link, child alars_module_base_link, origin xyz=0 0 0 rpy=0 0 0
- added joint fisheye_camera_joint: type fixed, parent fisheye_base_link, child fisheye_camera_link, origin xyz=0 0 0.016 rpy=3.14 -1.57 0
- joint fisheye_base_joint: parent module_base_link -> alars_module_base_link
- joint gimbal_base_joint: parent module_base_link -> alars_module_base_link
- joint rope_base_joint: parent module_base_link -> alars_module_base_link

Commit message: alars.urdf: fisheye_optical_frame"

File: vehicles/descriptions/alars_description/urdf/alars.urdf (robot description, URDF)
Before this commit: robot alars, 6 links, 5 joints
Links:
- added link fisheye_optical_frame
Joints:
- added joint fisheye_optical_joint: type fixed, parent fisheye_camera_link, child fisheye_optical_frame, origin xyz=0 0 0 rpy=-1.57 0 -1.57
