Commit message: alars:fc30, m350 urdfs. removed fisheye for now...

File: vehicles/descriptions/alars_description/urdf/M350.urdf (robot description, URDF)
Before this commit: robot alars, 7 links, 6 joints
Links:
- removed link fisheye_base_link
- removed link fisheye_camera_link
- removed link fisheye_optical_frame
Joints:
- removed joint fisheye_base_joint
- removed joint fisheye_camera_joint
- removed joint fisheye_optical_joint
- joint base_to_module_joint: origin xyz=0 0 0 rpy=0 0 0 -> xyz=0.00276 0 0.24600 rpy=0 0 0
- joint gimbal_base_joint: origin xyz=-0.082 0 -0.103 rpy=3.14 0 3.14 -> xyz=-0.07840 0 -0.13482 rpy=3.14 0 3.14
- joint rope_base_joint: origin xyz=0.10651 0 -0.12758 rpy=0 0 0 -> xyz=0.11005 0 -0.15937 rpy=0 0 0

Commit message: m350 urdf

File: vehicles/descriptions/alars_description/urdf/M350.urdf (robot description, URDF)
Before this commit: robot alars, 4 links, 3 joints
Links:
- added link landing_gear_center_link
Joints:
- removed joint base_to_module_joint
- added joint base_to_landing_gear_center: type fixed, parent base_link, child landing_gear_center_link, origin xyz=0.056 0 -0.335 rpy=0 0 0
- added joint landing_gear_center_to_module_joint: type fixed, parent landing_gear_center_link, child alars_module_base_link, origin xyz=0.00276 0 0.24600 rpy=0 0 0
