Commit message: fc30 urdf

File: vehicles/descriptions/alars_description/urdf/FC30.urdf (robot description, URDF)
Before this commit: robot alars, 4 links, 3 joints
Links:
- added link landing_gear_center_link
Joints:
- removed joint base_to_module_joint
- added joint base_to_landing_gear_center: type fixed, parent base_link, child landing_gear_center_link, origin xyz=0 0 -0.54231 rpy=0 0 0
- added joint landing_gear_center_to_module_joint: type fixed, parent landing_gear_center_link, child alars_module_base_link, origin xyz=0.35363 0 0.22881 rpy=0 0 -1.57
- joint rope_base_joint: parent base_link -> landing_gear_center_link
