Commit message: Changes in evolo launch file and evolo description

File: vehicles/descriptions/evolo_description/urdf/evolo.urdf (robot description, URDF)
Before this commit: robot evolo, 6 links, 5 joints
Links:
- removed link evolo/camera_link
- added link evolo/gimbalz1_base
Joints:
- joint evolo/camera_joint: child evolo/camera_link -> evolo/gimbalz1_base; origin xyz=-0.1 0.1 0.05 rpy=0 0 0 -> xyz=0.7 0.0 0.15 rpy=0 0 0
- joint evolo/lidar_joint: origin xyz=0.1 0.1 0 rpy=0 0 0 -> xyz=0.83 0.0 0.1 rpy=0 0 0

Commit message: update evolo's camera link name in urdf

File: vehicles/descriptions/evolo_description/urdf/evolo.urdf (robot description, URDF)
Before this commit: robot evolo, 6 links, 5 joints
Links:
- removed link evolo/gimbalz1_base
- added link evolo/gimbal/z1_base
Joints:
- joint evolo/camera_joint: child evolo/gimbalz1_base -> evolo/gimbal/z1_base
