Commit message: changed urdf

File: vehicles/descriptions/evolo_description/urdf/evolo.urdf (robot description, URDF)
Before this commit: robot evolo, 6 links, 5 joints
Joints:
- joint evolo/camera_joint: origin xyz=0.7 0.0 0.15 rpy=0 0 0 -> xyz=--0.4 0.0 1.0 rpy=0 0 0
- joint evolo/lidar_joint: origin xyz=0.83 0.0 0.1 rpy=0 0 0 -> xyz=0.35 0.0 0.27 rpy=0 0 0
- joint sensor_imu_joint: origin xyz=-0.002 -0.010 0.008 rpy=0 0 0 -> xyz=-0.002 -0.010 0.008 rpy=0 0 0.7853981633974483
- joint sensor_lidar_joint: origin xyz=0 0 0.038 rpy=0 0 3.141592653589793 -> xyz=0 0 0.038 rpy=0 0 2.356194490192345

Commit message: removed -

File: vehicles/descriptions/evolo_description/urdf/evolo.urdf (robot description, URDF)
Before this commit: robot evolo, 6 links, 5 joints
Joints:
- joint evolo/camera_joint: origin xyz=--0.4 0.0 1.0 rpy=0 0 0 -> xyz=-0.4 0.0 1.0 rpy=0 0 0

Commit message: changed urdf again

File: vehicles/descriptions/evolo_description/urdf/evolo.urdf (robot description, URDF)
Before this commit: robot evolo, 6 links, 5 joints
Joints:
- joint evolo/lidar_joint: origin xyz=0.35 0.0 0.27 rpy=0 0 0 -> xyz=0.35 0.0 0.27 rpy=0 0 1.57079633
- joint sensor_lidar_joint: origin xyz=0 0 0.038 rpy=0 0 2.356194490192345 -> xyz=0 0 0.038 rpy=0 0 3.141592653589793
